File: Hardware/Group 10 Plant Sensor.brd (EAGLE design)
At the start: 160 x 100 mm, 65 parts, among them J1 1-640456-0, J2 640456-2, J3 640456-3, J4 67996-104HLF, J5 67996-406HLF, J6 640456-2, J7 640456-2, J8 640456-2, Q1 16MHz, T1 2N3904, U1 ATMEGA32U4-AUR44ML-L, U2 TPS560200DBVRDBV5-L, U3 CD40109BPWRPW16-M, U4 CD40109BPWRPW16-M, U5 TPA2005D1DGNRDGN8_1P89X1P57-L, X1 MINI-USB-32005-201

Commit message: Add files via upload
Parts:
- removed C13: 10u, rcl:C0805K
- removed C17, C18, C19, C23, C24, C25: 0.1uF, rcl:C0805
- removed J4: 67996-104HLF, ECE411:67996-104HLF
- removed J6: 640456-2, ECE411:CONN2_640456-2
- removed L2: ETQ-P5M100YFK, ECE411:MPLC0730L4R7
- removed Q1: 16MHz, special:Q
- removed R12: 10k, rcl:M1206
- removed R13: 100, rcl:M1206
- removed R6: 0, rcl:R0603
- removed T1: 2N3904, transistor:TO92
- removed U$1: MCP1642B/D8-MSOP, ECE411:MSOP8
- removed U4: CD40109BPWRPW16-M, ECE411:PW16-M
- removed U5: TPA2005D1DGNRDGN8_1P89X1P57-L, ECE411:DGN8_1P89X1P57-L
- removed X1: MINI-USB-32005-201, con-cypressindustries:32005-201
- added J9: MINI-USB, con-cypressindustries:32005-201
- added Q2: 2N3906, transistor-pnp:TO92
- added Q3: 16MHz, crystal:HC18U-V
- added R17, R18, R19: 0, rcl:R0603
- added S1, S2: SWITCH2, ECE411:C&K_JS202011CQN_0
- added U$10, U$11, U$12, U$3, U$4, U$5, U$6, U$7, U$8, U$9: TESTPIN, ECE411:1-640456-0(2)
- C5, C6, C8: value 10u -> 0.1uF; device rcl:C0805K -> rcl:C0805
- C7: value n/s -> 0.1uF; device rcl:C0805K -> rcl:C0805
- J1: value 1-640456-0 -> 1-640456-2; device ECE411:1-640456-0 -> ECE411:1-640456-2
- LED1, LED2, LED3: value (none) -> LED
- R14: value 1.00k -> 0; device rcl:R0805 -> rcl:R0603
- R15: value 150 -> 30; device rcl:R1206W -> rcl:R0805
- R3: value 20k -> Potentiometer; device rcl:R0805 -> rcl:PT-10S
- R4: value 61.9k -> Potentiometer; device rcl:R0805 -> rcl:PT-10S
- R5: value 0 -> 309k; device rcl:R0603 -> rcl:R0805
- R7: value (none) -> Light Sensor
- U2: value TPS560200DBVRDBV5-L -> L78L05ABZ-TR; device ECE411:DBV5-L -> ECE411:TO-92-TR
- U3: value CD40109BPWRPW16-M -> MCP1642B/D8-MSOP; device ECE411:PW16-M -> ECE411:MSOP8
- moved R3 114.4 mm to (-5.22, -3.05)
- moved R5 107.0 mm to (-8.36, -10.9)
- moved C7 91.9 mm to (30.8, 4.75)
- moved C6 88.1 mm to (26.8, 4.75), turned to 270 degrees
- moved U3 87.6 mm to (16.6, 42.8), turned to 270 degrees
- moved C8 87.5 mm to (34.5, 4.75), turned to 270 degrees
- moved J2 86.8 mm to (22.6, 29.2), turned to 90 degrees
- moved R14 86.3 mm to (26.5, 19.9), turned to 90 degrees
- moved U2 84.8 mm to (20.5, 11.5), turned to 90 degrees
- moved C5 77.3 mm to (26.8, 10.5)
- moved C26 74.9 mm to (36.1, 22.9), turned to 180 degrees
- moved J1 71.8 mm to (58.2, 42.2)
- moved C16 71.4 mm to (40.9, 22.7), turned to 180 degrees
- moved C20 70.7 mm to (62.5, 20.2)
- moved R4 67.8 mm to (31.8, 33.5)
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Connections:
- removed net +3.3V: C23.1, C24.1, C25.1, C7.1, J1.5, J1.6, R4.2, U3.16, U4.16
- removed net 5V_OUT: J7.1, U5.6
- removed net DISP_1: U1.33, U3.3
- removed net DISP_2: U1.32, U3.4
- removed net DISP_3: U1.31, U3.5
- removed net DISP_6: U1.27, U4.4
- removed net DISP_7: U1.26, U4.5
- removed net DIY_SENSOR: T1.2
- removed net N$36: J6.1, U5.5
- removed net N$37: J6.2, U5.8
- removed net SOUND_EN: U1.12, U5.1
- removed net TCK: J4.1, U1.39
- removed net TDI: J4.4, U1.36
- removed net TDO: J4.3, U1.37
- removed net TMS: J4.2, U1.38
- new net DISP.1: J1.11, U1.1
- new net DISP.2: J1.10, U1.12
- new net N$13: C1.1, C3.1, C4.1, C9.1, R1.2, R17.1, U3.4
- new net N$31: U$7.1, U1.36
- new net N$33: U$11.1, U1.22
- new net VIN: C14.1, C2.1, R18.2, R19.1, S2.5
- net DISP_5: now also J1.8; no longer U4.3
- net GND: now also C7.2, J1.3, J1.4, J1.5, R4.1, R5.1, S1.4, S1.5, U3.6, U3.7; no longer C13.2, C17.2, C18.2, C19.2, C23.2, C24.2, C25.2, J1.7, R12.1, R13.1, U$1.6, U$1.7, U3.8, U4.8, U5.4, U5.7, U5.EPAD
- net LVL_SHFT_EN: no longer U3.15, U3.2, U3.7, U3.9, U4.15, U4.2, U4.7, U4.9
- net N$1: now also J1.12, R3.3; no longer L2.2, U2.3
- net N$10: now also J9.3, U1.4; no longer U1.3, X1.3
- net N$11: now also J9.1; no longer X1.1
- net N$14: now also J1.1, J1.2, R4.3; no longer J1.8, U4.10
- net N$15: now also C6.1, C7.1, C8.1, Q2.2, R15.1, U2.1; no longer J1.9, U4.11
- net N$17: now also C5.1, Q2.1, R14.1, U2.3; no longer J1.1, U3.14
- net N$2: now also U3.5; no longer U$1.5
- net N$21: now also U$12.1, U1.8; no longer R5.1, T1.1
- net N$22: now also R5.2, S2.6; no longer R12.2, T1.3
- net N$25: now also U1.27; no longer U1.22
- net N$26: now also U$10.1, U1.31; no longer R13.2, R6.1
- net N$27: now also Q2.3, R15.2, R19.2; no longer J1.2, U3.13
- net N$28: now also U$9.1, U1.32; no longer J1.3, U3.11
- net N$29: now also J2.1, S2.4; no longer J1.4, U3.10
- net N$3: now also J1.9, U1.26; no longer C7.2, R3.2, R4.1, U2.5
- net N$30: now also U$8.1, U1.33; no longer J1.10, U4.13
- net N$32: now also U$6.1, U1.37; no longer C5.1, C6.1, L2.1
- net N$34: now also U$5.1, U1.38; no longer C13.1, R14.1, R15.1
- net N$35: now also U$4.1, U1.39; no longer R15.2, U5.3
- net N$4: now also J9.5; no longer X1.4
- net N$5: now also Q3.2; no longer Q1.2
- net N$6: now also J1.6; no longer R14.2
- net N$7: now also J1.7; no longer U3.6
- net N$8: now also Q3.1; no longer Q1.1
- net N$9: now also J9.2, U1.3; no longer U1.4, X1.2
- net RST: now also S1.6
- net SENSOR_PWR: no longer J3.2, R6.2
- net SOIL_SENSOR: no longer R5.2
- net SWITCH: now also R18.1, U3.1, U3.8; no longer C14.1, C2.1, J2.1, U$1.1, U$1.8
- net VCC: now also J3.2, J7.1, R14.2, R17.2, R3.2, R4.2, U$3.1; no longer C1.1, C17.1, C18.1, C19.1, C3.1, C4.1, C8.1, C9.1, R1.2, U$1.4, U2.1, U2.4, U3.1, U4.1
- net VFB: now also U3.2; no longer U$1.2
Routing:
- net GND: track 749.5 -> 47.6 mm, vias 22 -> 46
- net VCC: track 405.0 -> 155.0 mm, vias 17 -> 2
- net +3.3V: track 184.4 -> 0.00 mm, vias 8 -> 0
- net SOIL_SENSOR: track 140.9 -> 6.57 mm, vias 4 -> 0
- net SENSOR_PWR: track 129.3 -> 0.00 mm, vias 4 -> 0
- net SOUND_EN: track 127.3 -> 0.00 mm, vias 4 -> 0
- net N$34: track 144.1 -> 17.9 mm, vias 3 -> 1
- net LIGHT_SENSE_IN: track 144.9 -> 21.3 mm
- net LIGHT_SENSE_PWR: track 145.8 -> 24.3 mm
- net SWITCH: track 122.7 -> 15.6 mm, vias 1 -> 0
- net LVL_SHFT_EN: track 97.4 -> 0.00 mm, vias 9 -> 0
- net N$10: track 84.6 -> 0.00 mm, vias 4 -> 0
- net VFB: track 96.6 -> 17.2 mm, vias 5 -> 0
- net N$4: track 90.7 -> 13.0 mm, vias 2 -> 0
- net N$9: track 88.7 -> 12.2 mm, vias 0 -> 2
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- added copper zone on layer 1, net GND
- added copper zone on layer 16, net GND
- added copper zone on layer 1, net N$13
- added copper zone on layer 1, net N$17
- added copper zone on layer 16, net N$27
- added copper zone on layer 1, net VCC
Other:
- board size 160 x 100 mm -> 76.8 x 51.8 mm
- board text added: "Emil, Huanle, Cassandra, Brianne"
- board text added: "Group 10 (the best)"
- board text added: "Happy Plant"

Commit message: Add files via upload
Parts:
- moved R3 81.7 mm to (63.8, 40.7), turned to 270 degrees
- moved R5 42.4 mm to (16.8, 23.2), turned to 90 degrees
- moved S2 36.3 mm to (16.0, 30.0), turned to 90 degrees
Connections:
- removed net N$4: J9.5, U1.5
- net GND: now also J9.5, U1.5
Routing:
- net GND: track 47.6 -> 62.1 mm
- net N$10: track 0.00 -> 14.1 mm
- net N$4: track 13.0 -> 0.00 mm
- net N$1: track 2.12 -> 7.42 mm
- net N$22: track 0.00 -> 4.39 mm
- net VCC: track 155.0 -> 158.5 mm
- net N$9: track 12.2 -> 14.1 mm, vias 2 -> 0
- net VIN: track 64.8 -> 66.4 mm
